File: kiCAD/Multiplier.kicad_sch (KiCad schematic)
At the start: 58 parts, among them IC2 ADG1221BRMZ, J1 Conn_01x02_Pin, J2 Conn_01x02_Pin, J3 Conn_01x02_Pin, Q7 Q_Dual_PNP_PNP_C1B1B2C2E2E1, Q8 Q_Dual_PNP_PNP_C1B1B2C2E2E1, U1 TS912, U10 TPS63060, U2 TLV340, U4 TS912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

Commit message: Modified: Multiplier.kicad_pcb, added: backups files
Parts:
- R6: value 10k -> 2k
Changed lines of the file:
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@@
       (effects (font (size 1.27 1.27)) (justify right))
     )
-    (property "Value" "10k" (at 110.49 64.77 0)
+    (property "Value" "2k" (at 110.49 64.77 0)
       (effects (font (size 1.27 1.27)) (justify right))
     )
